Commit message: Test

File: description/gazebo_control.xacro (robot description, xacro)
@@ -9,5 +9,4 @@
             <wheel_radius>0.1</wheel_radius>
             <!-- Limits -->
-            <!-- <max_wheel_torque>200</max_wheel_torque> -->
             <max_linear_acceleration>10.0</max_linear_acceleration>
             <!-- Input -->

File: description/robot.urdf.xacro (robot description, xacro)
@@ -3,3 +3,4 @@
     <xacro:include filename="robot_core.xacro" />
     <xacro:include filename="gazebo_control.xacro"/>
+    <xacro:include filename="lidar.xacro" />
 </robot>

File: description/robot_core.xacro (robot description, xacro)
@@ -13,4 +13,7 @@
     <material name="black">
         <color rgba="0 0 0 1"/>
+    </material>
+    <material name="red">
+        <color rgba="1 0 0 1"/>
     </material>
     <!--  BASE LINK-->
@@ -43,57 +46,46 @@
     <gazebo reference="chassis">
         <material>Gazebo/White</material>
+        <mu1>0.2</mu1>
+        <mu2>0.2</mu2>
     </gazebo>
+    <xacro:macro name="wheel" params="prefix">
+        <link name="${prefix}_wheel">
+            <visual>
+                <geometry>
+                    <cylinder length="0.04" radius="0.05" />
+                </geometry>
+                <material name="blue"/>
+            </visual>
+            <collision>
+                <geometry>
+                    <cylinder length="0.04" radius="0.05" />
+                </geometry>
+            </collision>
+            <xacro:inertial_cylinder mass="0.1" length="0.04" radius="0.05" >
+                <origin xyz="0 0 0" rpy="0 0 0"/>
+            </xacro:inertial_cylinder>
+        </link>
+        <gazebo reference="${prefix}_wheel">
+            <mu1>0.2</mu1>
+            <mu2>0.2</mu2>
+            <material>Gazebo/Blue</material>
+        </gazebo>
+    </xacro:macro>
     <!-- LEFT WHEEL -->
     <joint name="left_wheel_joint" type="continuous">
-        <parent link="base_link"/>
-        <child link="left_wheel"/>
-        <origin xyz="0 0.175 0" rpy="-${pi/2} 0 0"/>
-        <axis xyz="0 0 1"/>
-    </joint>
-    <link name="left_wheel">
-        <visual>
-            <geometry>
-                <cylinder length="0.04" radius="0.05" />
-            </geometry>
-            <material name="blue"/>
-        </visual>
-        <collision>
-            <geometry>
-                <cylinder length="0.04" radius="0.05" />
-            </geometry>
-        </collision>
-        <xacro:inertial_cylinder mass="0.1" length="0.04" radius="0.05" >
-            <origin xyz="0 0 0" rpy="0 0 0"/>
-        </xacro:inertial_cylinder>
-    </link>
-    <gazebo reference="left_wheel">
-        <material>Gazebo/Blue</material>
-    </gazebo>
+            <parent link="base_link"/>
+            <child link="left_wheel"/>
+            <origin xyz="0 0.175 0" rpy="-${pi/2} 0 0"/>
+            <axis xyz="0 0 1"/>
+        </joint>
+    <xacro:wheel prefix="left" />
     <!-- RIGHT WHEEL -->
     <joint name="right_wheel_joint" type="continuous">
-        <parent link="base_link"/>
-        <child link="right_wheel"/>
-        <origin xyz="0 -0.175 0" rpy="${pi/2} 0 0"/>
-        <axis xyz="0 0 -1"/>
-    </joint>
-    <link name="right_wheel">
-        <visual>
-            <geometry>
-                <cylinder length="0.04" radius="0.05" />
-            </geometry>
-            <material name="blue"/>
-        </visual>
-        <collision>
-            <geometry>
-                <cylinder length="0.04" radius="0.05" />
-            </geometry>
-        </collision>
-        <xacro:inertial_cylinder mass="0.1" length="0.04" radius="0.05" >
-            <origin xyz="0 0 0" rpy="0 0 0"/>
-        </xacro:inertial_cylinder>
-    </link>
-    <gazebo reference="right_wheel">
-        <material>Gazebo/Blue</material>
-    </gazebo>
+            <parent link="base_link"/>
+            <child link="right_wheel"/>
+            <origin xyz="0 -0.175 0" rpy="${pi/2} 0 0"/>
+            <axis xyz="0 0 -1"/>
+        </joint>
+    <xacro:wheel prefix="right" />
     <!-- CASTER WHEEL -->
     <joint name="caster_wheel_joint" type="fixed">
@@ -119,4 +111,6 @@
     </link>
     <gazebo reference="caster_wheel">
+        <mu1>0.0000002</mu1>
+        <mu2>0.0000002</mu2>
         <material>Gazebo/Black</material>
     </gazebo>

Commit message: Versione Finale del Progetto
Vengono sostituiti tutti i precedenti file

File: description/gazebo_control.xacro (robot description, xacro)
@@ -6,8 +6,8 @@
             <left_joint>left_wheel_joint</left_joint>
             <right_joint>right_wheel_joint</right_joint>
-            <wheel_separation>0.35</wheel_separation>
-            <wheel_radius>0.1</wheel_radius>
+            <wheel_separation>0.297</wheel_separation>
+            <wheel_radius>0.06</wheel_radius>
             <!-- Limits -->
-            <max_linear_acceleration>10.0</max_linear_acceleration>
+            <max_linear_acceleration>10</max_linear_acceleration>
             <!-- Input -->
             <topic>cmd_vel</topic>

File: description/lidar.xacro (robot description, xacro)
@@ -4,5 +4,5 @@
         <parent link="chassis"/>
         <child link="laser_frame"/>
-        <origin xyz="0.122 0 0.212" rpy="0 0 0"/>
+        <origin xyz="0.122 0 0.2" rpy="0 0 0"/>
     </joint>
     <link name="laser_frame">
@@ -25,5 +25,5 @@
             </geometry>
         </collision>
-        <xacro:inertial_cylinder mass="0.1" length="0.04" radius="0.05">
+        <xacro:inertial_cylinder mass="0.05" length="0.04" radius="0.05">
             <origin xyz="0 0 0" rpy="0 0 0"/>
         </xacro:inertial_cylinder>
@@ -35,7 +35,6 @@
             <pose> 0 0 0 0 0 0 </pose>
             <visualize>true</visualize>
-            <update_rate>5</update_rate>
-            <topic>scan</topic>
-            <gz_frame_id>laser_frame</gz_frame_id>
+            <update_rate>30</update_rate>
+            <topic>laser_scan</topic>
             <lidar>
                 <scan>
@@ -53,4 +52,5 @@
                 </range>
             </lidar>
+            <gz_frame_id>laser_frame</gz_frame_id>
         </sensor>
     </gazebo>

File: description/robot_core.xacro (robot description, xacro)
@@ -2,4 +2,5 @@
 <robot xmlns:xacro="http://www.ros.org/wiki/xacro"  name="robot">
     <xacro:include filename="inertial_macros.xacro"/>
+    <!-- Color def -->
     <material name="white">
         <color rgba="1 1 1 1" />
@@ -17,4 +18,19 @@
         <color rgba="1 0 0 1"/>
     </material>
+    <!--Structure data-->
+    <xacro:property name="chassis_mass" value="10.0"/>
+    <xacro:property name="chassis_lenght" value="0.335"/>
+    <xacro:property name="chassis_width" value="0.265"/>
+    <xacro:property name="chassis_height" value="0.1"/>
+    <xacro:property name="wheel_mass" value="0.5"/>
+    <xacro:property name="wheel_radius" value="0.06"/>
+    <xacro:property name="wheel_thickness" value="0.026"/>
+    <xacro:property name="wheel_position_x" value="0.226"/>
+    <xacro:property name="wheel_position_y" value="0.1485"/>
+    <xacro:property name="wheel_position_z" value="0.01"/>
+    <xacro:property name="caster_wheel_mass" value="0.05"/>
+    <xacro:property name="caster_wheel_radius" value="0.08" />
+    <xacro:property name="caster_wheel_position_x" value="0.1"/>
+    <xacro:property name="caster_wheel_position_z" value="${caster_wheel_radius - wheel_radius - wheel_position_z}"/>
     <!--  BASE LINK-->
     <link name="base_link">
@@ -24,28 +40,26 @@
         <parent link="base_link"/>
         <child link="chassis"/>
-        <origin xyz="-0.1 0 0"/>
+        <origin xyz="${-wheel_position_x} 0 ${wheel_position_z}"/>
     </joint>
     <link name="chassis">
         <visual>
-            <origin xyz="0.15 0 0.075" rpy="0 0 0"/>
+            <origin xyz="${chassis_lenght/2} 0 ${chassis_height/2}" rpy="0 0 0"/>
             <geometry>
-                <box size="0.3 0.3 0.15"/>
+                <box size="${chassis_lenght} ${chassis_width} ${chassis_height}"/>
             </geometry>
             <material name="white"/>
         </visual>
         <collision>
-            <origin xyz="0.15 0 0.075" rpy="0 0 0"/>
+            <origin xyz="${chassis_lenght/2} 0 ${chassis_height/2}" rpy="0 0 0"/>
             <geometry>
-                <box size="0.3 0.3 0.15"/>
+                <box size="${chassis_lenght} ${chassis_width} ${chassis_height}"/>
             </geometry>
         </collision>
-        <xacro:inertial_box mass="0.5" x="0.3" y="0.3" z="0.15">
-            <origin xyz="0.15 0 0.075" rpy ="0 0 0"/>
+        <xacro:inertial_box mass="${chassis_mass}" x="${chassis_lenght}" y="${chassis_width}" z="${chassis_height}">
+            <origin xyz="${chassis_lenght/2} 0 ${chassis_height/2}" rpy ="0 0 0"/>
         </xacro:inertial_box>
     </link>
     <gazebo reference="chassis">
         <material>Gazebo/White</material>
-        <mu1>0.2</mu1>
-        <mu2>0.2</mu2>
     </gazebo>
     <xacro:macro name="wheel" params="prefix">
@@ -53,5 +67,5 @@
             <visual>
                 <geometry>
-                    <cylinder length="0.04" radius="0.05" />
+                    <cylinder length="${wheel_thickness}" radius="${wheel_radius}" />
                 </geometry>
                 <material name="blue"/>
@@ -59,8 +73,8 @@
             <collision>
                 <geometry>
-                    <cylinder length="0.04" radius="0.05" />
+                    <sphere radius="${wheel_radius}" />
                 </geometry>
             </collision>
-            <xacro:inertial_cylinder mass="0.1" length="0.04" radius="0.05" >
+            <xacro:inertial_cylinder mass="${wheel_mass}" length="${wheel_thickness}" radius="${wheel_radius}" >
                 <origin xyz="0 0 0" rpy="0 0 0"/>
             </xacro:inertial_cylinder>
@@ -76,7 +90,9 @@
             <parent link="base_link"/>
             <child link="left_wheel"/>
-            <origin xyz="0 0.175 0" rpy="-${pi/2} 0 0"/>
+            <origin xyz="0 ${wheel_position_y} 0" rpy="-${pi/2} 0 0"/>
             <axis xyz="0 0 1"/>
-        </joint>
+            <dynamics damping="10000.0" friction="1000.0"/>
+            <limit effort="10000" velocity="10"/>
+    </joint>
     <xacro:wheel prefix="left" />
     <!-- RIGHT WHEEL -->
@@ -84,7 +100,9 @@
             <parent link="base_link"/>
             <child link="right_wheel"/>
-            <origin xyz="0 -0.175 0" rpy="${pi/2} 0 0"/>
+            <origin xyz="0 ${-wheel_position_y} 0" rpy="${pi/2} 0 0"/>
             <axis xyz="0 0 -1"/>
-        </joint>
+            <dynamics damping="10000.0" friction="1000.0"/>
+            <limit effort="10000" velocity="10"/>
+    </joint>
     <xacro:wheel prefix="right" />
     <!-- CASTER WHEEL -->
@@ -92,10 +110,10 @@
         <parent link="chassis"/>
         <child link="caster_wheel"/>
-        <origin xyz="0.24 0 0"/>
+        <origin xyz="${caster_wheel_position_x} 0 ${caster_wheel_position_z}"/>
     </joint>
     <link name="caster_wheel">
         <visual>
             <geometry>
-                <sphere radius="0.05"/>
+                <sphere radius="${caster_wheel_radius}"/>
             </geometry>
             <material name="black"/>
@@ -103,14 +121,14 @@
         <collision>
             <geometry>
-                <sphere radius="0.05"/>
+                <sphere radius="${caster_wheel_radius}"/>
             </geometry>
         </collision>
-        <xacro:inertial_sphere mass="0.1" radius="0.05">
+        <xacro:inertial_sphere mass="${caster_wheel_mass}" radius="${caster_wheel_radius}">
             <origin xyz="0 0 0" rpy="0 0 0"/>
         </xacro:inertial_sphere>
     </link>
     <gazebo reference="caster_wheel">
-        <mu1>0.0000002</mu1>
-        <mu2>0.0000002</mu2>
+        <mu1>0.02</mu1>
+        <mu2>0.02</mu2>
         <material>Gazebo/Black</material>
     </gazebo>
